File: hardware/Bsides_2024_Guest/Bsides_2024_Guest.kicad_pcb (KiCad board)
At the start: 2 copper layers, 134.5 x 127.4 mm, 45 parts, among them J1 Conn_02x03_Odd_Even, J2 Battery, J3 Battery, J4 OLED, J5 Conn_01x05, J6 Conn_01x05, P1 USB_C_Plug_USB2.0, Q1 DMG3415U-7, SW1 ON, SW2 RESET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

Commit message: feat(Hw): Update PCB
Parts:
- J4: moved to F.Cu
- moved J4 41.5 mm to (69.1, 124.0)
- moved R6 9.67 mm to (76.8, 139.3)
- moved D2 8.99 mm to (80.1, 136.6)
- moved C5 8.61 mm to (76.2, 136.4)

Commit message: feat(Hw): Update PCB and schematic
Parts:
- removed the Ref** at (125.5, 89.8)
- added Ref**: Val**, Guest:Badge_Guest_Bsides_2024_CDMX (1), F.Cu at (125.1, 89.3)
- J1: value Conn_02x03_Odd_Even -> Add_On
- moved C7 2.02 mm to (103.2, 40.5)
- moved D4 2.02 mm to (106.7, 40.4)
- moved C12 1.47 mm to (147.4, 40.4)
- moved D5 1.47 mm to (150.9, 40.7)
- moved J1 0.98 mm to (148.2, 75.9)
- moved J5 0.11 mm to (186.8, 140.1), turned to -43.926 degrees
- moved J6 0.07 mm to (64.4, 135.4), turned to 45.111 degrees
Connections:
- C1 pad 1: Net-(SW1-B) -> VBUS
- C12 pad 2: +3V3 -> /VOUT
- C13 pad 1: +3V3 -> /VOUT
- C14 pad 1: +3V3 -> /VOUT
- C15 pad 1: +3V3 -> /VOUT
- C2 pad 1: +3V3 -> Net-(D1-A)
- C5 pad 2: +3V3 -> /VOUT
- C6 pad 2: +3V3 -> /VOUT
- C7 pad 2: +3V3 -> /VOUT
- D1 pad 2: VBUS -> Net-(D1-A)
- D2 pad 1: +3V3 -> /VOUT
- D3 pad 1: +3V3 -> /VOUT
- D4 pad 1: +3V3 -> /VOUT
- D5 pad 1: +3V3 -> /VOUT
- J1 pad 1: unconnected-(J1-Pin_1-Pad1) -> /VOUT
- J1 pad 2: unconnected-(J1-Pin_2-Pad2) -> GND
- J1 pad 3: unconnected-(J1-Pin_3-Pad3) -> /SDA
- J1 pad 4: unconnected-(J1-Pin_4-Pad4) -> /SCL
- J4 pad 1: +3V3 -> /VOUT
- Q1 pad 1: VBUS -> Net-(D1-A)
- R1 pad 2: +3V3 -> /VOUT
- R2 pad 1: VBUS -> Net-(D1-A)
- R5 pad 2: +3V3 -> /VOUT
- SW1 pad 2: Net-(SW1-B) -> /VOUT
- U1 pad 2: +3V3 -> /VOUT
- U2 pad 1: Net-(SW1-B) -> VBUS
- U2 pad 3: Net-(SW1-B) -> VBUS
- U2 pad 5: +3V3 -> Net-(D1-A)
Routing:
- added copper zone on F.Cu, net GND
Other:
- board size 134.5 x 127.4 mm -> 134.5 x 129.5 mm
