File: hardware/Bsides_2024_Guest/Bsides_2024_Guest.kicad_sch (KiCad schematic)
At the start: 44 parts, among them J1 Add_On, J2 Battery, J3 Battery, J4 OLED, J5 Serial_IN, J6 Serial_OUT, P1 USB_C_Plug_USB2.0, Q1 DMG3415U-7, SW1 ON, SW2 RESET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

Commit message: feat(Hw): Update route
Parts:
- C10, C11, C8, C9: LCSC# (none) -> C478888
- C12, C5, C6, C7: LCSC# C42998 -> C478888; manf# 0603F104M500NT -> (none)
Changed lines of the file:
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@@
 			)
 		)
-		(property "Datasheet" "~"
+		(property "Datasheet" ""
 			(at 249.428 119.761 0)
 			(effects
@@
 			)
 		)
-		(property "LCSC#" "C42998"
+		(property "LCSC#" "C478888"
 			(at 249.428 119.761 0)
 			(effects
@@
 			)
 		)
-		(property "manf#" "0603F104M500NT"
+		(property "manf#" ""
 			(at 249.428 119.761 0)
 			(effects
@@
 			)
 		)
-		(property "Datasheet" "~https://datasheet.lcsc.com/lcsc/1811021421_Samsung-Electro-Mechanics-CL10A106MP8NNNC_C85713.pdf"
+		(property "Datasheet" ""
 			(at 41.148 178.562 0)
 			(effects
@@
 			)
 		)
-		(property "Datasheet" "~"
+		(property "Datasheet" ""
 			(at 258.064 88.646 0)
 			(effects
@@
 			)
 		)
+		(property "LCSC#" "C478888"
+			(at 258.064 88.646 0)
+			(effects
+				(font
+					(size 1.27 1.27)
+				)
+				(hide yes)
+			)
+		)
 		(pin "2"
 		)
@@
 			)
 		)
-		(property "Datasheet" "~https://datasheet.lcsc.com/lcsc/1811021421_Samsung-Electro-Mechanics-CL10A106MP8NNNC_C85713.pdf"
+		(property "Datasheet" ""
 			(at 65.532 176.53 0)
 			(effects
@@
 			)
 		)
-		(property "Datasheet" "~"
+		(property "Datasheet" ""
 			(at 200.025 119.761 0)
 			(effects
@@
 			)
 		)
-		(property "LCSC#" "C42998"
+		(property "LCSC#" "C478888"
 			(at 200.025 119.761 0)
 			(effects
@@
 			)
 		)
-		(property "manf#" "0603F104M500NT"
+		(property "manf#" ""
 			(at 200.025 119.761 0)
 			(effects
@@
 			)
 		)
-		(property "Datasheet" "~"
+		(property "Datasheet" ""
 			(at 259.334 69.596 0)
 			(effects
@@
 			)
 		)
+		(property "LCSC#" "C478888"
+			(at 259.334 69.596 0)
+			(effects
+				(font
+					(size 1.27 1.27)
+				)
+				(hide yes)
+			)
+		)
 		(pin "2"
 		)
@@
 			)
 		)
-		(property "Datasheet" "https://datasheet.lcsc.com/lcsc/1912111437_CCTC-TCC0603COG100J500CT_C376764.pdf"
+		(property "Datasheet" ""
 			(at 193.04 54.61 0)
 			(effects
@@
 			)
 		)
-		(property "Datasheet" "~"
+		(property "Datasheet" ""
 			(at 224.917 119.761 0)
 			(effects
@@
 			)
 		)
-		(property "LCSC#" "C42998"
+		(property "LCSC#" "C478888"
 			(at 224.917 119.761 0)
 			(effects
@@
 			)
 		)
-		(property "manf#" "0603F104M500NT"
+		(property "manf#" ""
 			(at 224.917 119.761 0)
 			(effects
@@
 			)
 		)
-		(property "Datasheet" "~"
+		(property "Datasheet" ""
 			(at 259.334 32.766 0)
 			(effects
@@
 			)
 		)
+		(property "LCSC#" "C478888"
+			(at 259.334 32.766 0)
+			(effects
+				(font
+					(size 1.27 1.27)
+				)
+				(hide yes)
+			)
+		)
 		(pin "2"
 		)
@@
 			)
 		)
-		(property "Datasheet" "https://datasheet.lcsc.com/lcsc/1912111437_CCTC-TCC0603COG100J500CT_C376764.pdf"
+		(property "Datasheet" ""
 			(at 191.77 69.85 0)
 			(effects
@@
 			)
 		)
-		(property "Datasheet" "~"
+		(property "Datasheet" ""
 			(at 259.334 53.086 0)
 			(effects
@@
 			)
 		)
+		(property "LCSC#" "C478888"
+			(at 259.334 53.086 0)
+			(effects
+				(font
+					(size 1.27 1.27)
+				)
+				(hide yes)
+			)
+		)
 		(pin "2"
 		)
@@
 			)
 		)
-		(property "Datasheet" "~"
+		(property "Datasheet" ""
 			(at 274.32 119.761 0)
 			(effects
@@
 			)
 		)
-		(property "LCSC#" "C42998"
+		(property "LCSC#" "C478888"
 			(at 274.32 119.761 0)
 			(effects
@@
 			)
 		)
-		(property "manf#" "0603F104M500NT"
+		(property "manf#" ""
 			(at 274.32 119.761 0)
 			(effects
