File: hardware/Bsides_2024_Guest/Bsides_2024_Guest.kicad_sch (KiCad schematic)
At the start: 44 parts, among them J1 Add_On, J2 Battery, J3 Battery, J4 OLED, J5 Serial_IN, J6 Serial_OUT, P1 USB_C_Plug_USB2.0, Q1 DMG3415U-7, SW1 ON, SW2 RESET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

Commit message: feat(Hw):Update_BOM_Added_Labels
Parts:
- C1, C14, C15, C2: LCSC# C85713 -> C85713; Proveedor (none) -> JLCPCB; manf# (none) -> GRM188R61E106KA73J
- C10, C11, C3, C4, C8, C9: LCSC# C478888 -> C478888; Proveedor (none) -> JLCPCB; manf# (none) -> KAM15AR71C104KM
- C12, C5, C6, C7: LCSC# C478888 -> C478888; Proveedor LCSC -> JLCPCB; manf# (none) -> KAM15AR71C104KM
- C13: Proveedor (none) -> JLCPCB; manf# (none) -> TMK107BJ105KA8T
- D1, Q1: Proveedor (none) -> JLCPCB
- D2, D3, D4, D5: Proveedor LCSC -> JLCPCB
- F1: value 0.5A -> 0.75A; LCSC# - -> C1972808; Proveedor (none) -> JLCPCB; manf# MFU0805FF00500P100 -> MFU0805FF00750P100
- J1: LCSC# (none) -> C5116527; Proveedor (none) -> JLCPCB
- J2, J3: LCSC# C5290193 -> C5290181; Proveedor (none) -> JLCPCB
- J4: Proveedor (none) -> UNIT ELECTRONICS; manf# Display OLED 128×32 0.91 I2C SSD1306 Blanco / Azul -> Display OLED 128Ã—32 0.91 I2C SSD1306 Blanco / Azul
- J5: LCSC# (none) -> C5333416; Proveedor (none) -> JLCPCB
- J6: LCSC# (none) -> C5116529; Proveedor (none) -> JLCPCB
- P1: LCSC# C2987386 -> C393939; Proveedor (none) -> JLCPCB
- R1: LCSC# (none) -> C403480; Proveedor (none) -> JLCPCB; manf# (none) -> ERJ-3GEYJ332V
- R2: Proveedor LCSC -> JLCPCB; manf# (none) -> RC0603DR-07100KL
- R3, R4: LCSC# C191782 -> C113390; Proveedor (none) -> JLCPCB; manf# ERJ3RBD5101V -> AC0603DR-075K1L
- R5: Proveedor (none) -> JLCPCB; manf# CR-03JL7---10K -> RMC1/16K1002DTP
- R6: Proveedor (none) -> JLCPCB; manf# RTT03471JTP -> ERJ-3RBD4700V
- SW1: LCSC# - -> C431540; Proveedor (none) -> JLCPCB; manf# JS102011SAQN -> (none)
- SW2: value RESET -> ~; Proveedor (none) -> JLCPCB; manf# (none) -> TL3342F160QG
- SW3: value BOOT -> ~; Proveedor (none) -> JLCPCB; manf# (none) -> TL3342F160QG
- SW4, SW6: value RESET -> ~; LCSC# C2886897 -> C318889; Proveedor (none) -> JLCPCB; manf# (none) -> TL3342F160QG
- SW5, SW7: LCSC# C2886897 -> C318889; Proveedor (none) -> JLCPCB; manf# (none) -> TL3342F160QG
- U1: Proveedor (none) -> MOUSER; manf# ESP32-C6-WROOM-1U-N4 -> ESP32-C6-WROOM-1-N4
- U2: LCSC# C150742 -> C51118; Proveedor (none) -> JLCPCB; manf# AP7365-33WG-7 -> AP2112K3.3TRG

Commit message: feat(Hw):Update_Guest_SCH_Labels
Connections:
- net GPIO16 renamed TX
- net GPIO17 renamed RX
- net GPIO4 renamed RX1
- net GPIO5 renamed TX1
Changed lines of the file:
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@@
 		)
 	)
-	(label "GPIO17"
+	(label "RX"
 		(at 62.23 68.072 0)
 		(fields_autoplaced yes)
@@
 		)
 	)
-	(label "GPIO16"
+	(label "TX"
 		(at 62.23 65.278 0)
 		(fields_autoplaced yes)
@@
 		)
 	)
-	(label "GPIO5"
+	(label "TX1"
 		(at 136.652 120.65 0)
 		(fields_autoplaced yes)
@@
 		)
 	)
-	(label "GPIO16"
+	(label "TX"
 		(at 18.796 118.11 0)
 		(fields_autoplaced yes)
@@
 		)
 	)
-	(label "GPIO17"
+	(label "RX"
 		(at 18.796 120.65 0)
 		(fields_autoplaced yes)
@@
 		)
 	)
-	(label "GPIO5"
+	(label "TX1"
 		(at 27.686 43.434 0)
 		(fields_autoplaced yes)
@@
 		)
 	)
-	(label "GPIO4"
+	(label "RX1"
 		(at 27.686 40.386 0)
 		(fields_autoplaced yes)
@@
 		)
 	)
-	(label "GPIO4"
+	(label "RX1"
 		(at 136.652 118.11 0)
 		(fields_autoplaced yes)
