File: hardware/Bsides_2024_Speaker/Bsides_2024_Speaker.kicad_sch (KiCad schematic)
At the start: 44 parts, among them J1 Add_On, J2 Battery, J3 Battery, J4 OLED, J5 Serial_IN, J6 Serial_OUT, P1 USB_C_Plug_USB2.0, Q1 DMG3415U-7, SW1 ON, SW2 SW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

Commit message: Faet(Hw): Update BOM Speaker
Parts:
- J2, J3: LCSC# C5290193 -> C5290181; Proveedor JLCPCB -> JLCPCB y LCSC
- R6: Proveedor Mouser -> JLCPCB
- U2: LCSC# C3021085 -> C51118; Proveedor Mouser -> JLCPCB
Changed lines of the file:
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@@
 			)
 		)
-		(property "LCSC#" "C5290193"
+		(property "LCSC#" "C5290181"
 			(at 160.528 158.75 0)
 			(effects
@@
 			)
 		)
-		(property "Proveedor" "JLCPCB"
+		(property "Proveedor" "JLCPCB y LCSC"
 			(at 160.528 158.75 0)
 			(effects
@@
 			)
 		)
-		(property "LCSC#" "C3021085"
+		(property "LCSC#" "C51118"
 			(at 68.834 175.26 0)
 			(effects
@@
 			)
 		)
-		(property "Proveedor" "Mouser"
+		(property "Proveedor" "JLCPCB"
 			(at 68.834 175.26 0)
 			(effects
@@
 			)
 		)
-		(property "LCSC#" "C5290193"
+		(property "LCSC#" "C5290181"
 			(at 160.528 163.957 0)
 			(effects
@@
 			)
 		)
-		(property "Proveedor" "JLCPCB"
+		(property "Proveedor" "JLCPCB y LCSC"
 			(at 160.528 163.957 0)
 			(effects
@@
 			)
 		)
-		(property "Proveedor" "Mouser"
+		(property "Proveedor" "JLCPCB"
 			(at 179.324 130.048 0)
 			(effects
