File: hardware/Bsides_2024_Community/Bsides_2024_Community.kicad_sch (KiCad schematic)
At the start: 44 parts, among them J1 Add_On, J2 Battery, J3 Battery, J4 OLED, J5 Serial_IN, J6 Serial_OUT, P1 USB_C_Plug_USB2.0, Q1 DMG3415U-7, SW1 ON, SW2 RESET, SW3 BOOT, SW4 RESET, SW6 RESET, U1 ESP32-C6-WROOM-1U-N4, U2 AP2112K-3.3

Commit message: feat(Hw): Update BOM
Parts:
- C1, C13, C14, C15, C2, C3, C4, D1: Proveedor (none) -> JLCPCB
- C10, C11, C8, C9: LCSC# (none) -> C478888; Proveedor (none) -> JLCPCB
- C12, C5, C6, C7: LCSC# C42998 -> C478888; Proveedor LCSC -> JLCPCB; manf# 0603F104M500NT -> (none)
- D2, D3, D4, D5: Proveedor LCSC -> JLCPCB
- F1: value 0.5A -> 0.75A; LCSC# - -> C1972808; Proveedor (none) -> JLCPCB
- J1: LCSC# (none) -> C5116527; Proveedor (none) -> JLCPCB
- J2, J3: LCSC# C5290193 -> C5290181; Proveedor (none) -> JLCPCB y LCSC
- J4: Proveedor (none) -> UNIT ELECTRONICS
- J5: LCSC# (none) -> C5333416; Proveedor (none) -> JLCPCB
- J6: LCSC# (none) -> C5116529; Proveedor (none) -> JLCPCB
- P1: LCSC# C2987386 -> C393939; Proveedor (none) -> JLCPCB
- Q1: Proveedor (none) -> JLCPCB; manf# DMG3415U-7 -> DMG3415UQ-7
- R1: LCSC# (none) -> C403480; Proveedor (none) -> JLCPCB; manf# (none) -> ERJ-3GEYJ332V
- R2: Proveedor LCSC -> JLCPCB; manf# (none) -> RC0603DR-07100KL
- R3, R4: LCSC# C191782 -> C113390; Proveedor (none) -> JLCPCB; manf# ERJ3RBD5101V -> AC0603DR-075K1L
- R5: Proveedor (none) -> JLCPCB; manf# CR-03JL7---10K -> RMC1/16K1002DTP
- R6: Proveedor (none) -> JLCPCB; manf# RTT03471JTP -> ERJ-3RBD4700V
- SW1: LCSC# - -> C431540; Proveedor (none) -> JLCPCB; manf# JS102011SAQN -> (none)
- SW2, SW3: Proveedor (none) -> JLCPCB; manf# (none) -> TL3342F160QG
- SW4, SW6: value RESET -> ~; LCSC# C2886897 -> C318889; Proveedor (none) -> JLCPCB; manf# (none) -> TL3342F160QG
- SW5, SW7: LCSC# C2886897 -> C318889; Proveedor (none) -> JLCPCB; manf# (none) -> TL3342F160QG
- U1: Proveedor (none) -> MOUSER
- U2: LCSC# C150742 -> C51118; Proveedor (none) -> JLCPCB; manf# AP7365-33WG-7 -> AP2112K3.3TRG
