File: hardware/Bsides_2024_Community/Bsides_2024_Community.kicad_pcb (KiCad board)
At the start: 2 copper layers, 159.6 x 169.5 mm, 40 parts, among them J1 Conn_02x03_Odd_Even, J2 Battery, J3 Battery, J4 OLED, P1 USB_C_Plug_USB2.0, Q1 DMG3415U-7, SW1 ON, SW2 RESET, SW3 BOOT, SW4 RESET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

Commit message: feat(Hw): Start new floorplan
Parts:
- removed the Ref** at (145.8, 104.2)
- added Ref**: Val**, Community:Badge Community_Bsides 2024 CDMX, F.Cu at (136.2, 100.9)
- J1: moved to F.Cu
- J2, J3: footprint bsides:BH-AAA-A1aj001 -> Community:BATT_8BH-AA-A1AJ020_MYG
- moved C1 262.1 mm to (-69.4, 43.7)
- moved C12 262.1 mm to (-50.0, 90.3)
- moved C2 262.1 mm to (-75.0, 43.7)
- moved C3 262.1 mm to (-80.9, 22.2)
- moved C4 262.1 mm to (-139.5, 22.6)
- moved C5 262.1 mm to (-129.3, -19.3)
- moved C6 262.1 mm to (-85.5, -21.8)
- moved C7 262.1 mm to (-165.4, 106.8)
- moved D1 262.1 mm to (-65.4, 40.5)
- moved D2 262.1 mm to (-125.8, -19.5)
- moved D4 262.1 mm to (-162.0, 107.3)
- moved D5 262.1 mm to (-46.4, 90.2)
- moved Q1 262.1 mm to (-65.9, 45.7)
- moved R1 262.1 mm to (-116.3, 105.9)
- moved R2 262.1 mm to (-69.4, 40.7)
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Other:
- board size 159.6 x 169.5 mm -> 297.4 x 177.5 mm

Commit message: feat(Hw): Update PCB
Parts:
- added J5: Conn_01x05, Connector_PinHeader_2.54mm:PinHeader_1x05_P2.54mm_Vertical, F.Cu at (213.8, 147.4)
- added J6: Conn_01x05, Connector_PinHeader_2.54mm:PinHeader_1x05_P2.54mm_Vertical, F.Cu at (67.0, 165.1)
- moved C2 284.3 mm to (195.2, 132.2), turned to -52.6 degrees
- moved U2 283.5 mm to (197.8, 130.4), turned to -142.6 degrees
- moved C1 282.6 mm to (200.2, 128.7), turned to 127.4 degrees
- moved SW1 276.5 mm to (203.8, 123.9), turned to -52.6 degrees
- moved D1 276.0 mm to (197.0, 126.0), turned to 127.4 degrees
- moved R2 275.9 mm to (193.0, 125.8), turned to -142.6 degrees
- moved Q1 272.9 mm to (194.3, 128.2), turned to -142.6 degrees
- moved C4 260.8 mm to (96.4, 133.9), turned to -90 degrees
- moved R5 259.5 mm to (97.9, 133.9), turned to 90 degrees
- moved C12 255.5 mm to (200.1, 142.8)
- moved D5 255.5 mm to (203.7, 142.6)
- moved SW2 255.5 mm to (91.4, 133.9)
- moved C6 254.2 mm to (161.7, 37.5)
- moved D3 254.2 mm to (165.2, 38.0)
- moved C5 251.8 mm to (115.4, 40.0)
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Routing:
- net /D-: track 0.00 -> 103.1 mm
- net /D+: track 0.00 -> 102.7 mm
- net VBUS: track 0.00 -> 14.0 mm
- net Net-(D1-K): track 0.00 -> 10.3 mm, vias 0 -> 2
- net Net-(SW1-B): track 0.00 -> 10.3 mm
- net /EN: track 0.00 -> 10.1 mm
- net /GPIO23: track 0.00 -> 8.64 mm
- net /GPIO22: track 0.00 -> 8.63 mm
- net /GPIO15: track 0.00 -> 8.63 mm
- net /BOOT: track 0.00 -> 8.62 mm
- net /GPIO1: track 0.00 -> 8.60 mm
- net Net-(F1-Pad1): track 0.00 -> 3.36 mm
- net +3V3: track 0.00 -> 2.04 mm
Other:
- board size 297.4 x 177.5 mm -> 169.6 x 159.5 mm

Commit message: feat(Hw): Update PCB
Parts:
- J4: moved to F.Cu
- moved J4 99.8 mm to (72.3, 153.0), turned to 0 degrees
- moved D4 6.01 mm to (82.9, 165.3)
- moved C7 6.01 mm to (79.5, 164.8)
Other:
- outline, holes or cut-outs redrawn

Commit message: feat(Hw): Update PCB and schematic
Parts:
- added C13: 1uF, Capacitor_SMD:C_0603_1608Metric, B.Cu at (99.0, 90.5)
- added C14: 10uF, Capacitor_SMD:C_0603_1608Metric, B.Cu at (99.0, 93.0)
- added C15: 10uF, Capacitor_SMD:C_0603_1608Metric, B.Cu at (99.0, 95.5)
- J1: value Conn_02x03_Odd_Even -> Add_On
Connections:
- C1 pad 1: Net-(SW1-B) -> VBUS
- C12 pad 2: +3V3 -> /VOUT
- C2 pad 1: +3V3 -> Net-(D1-A)
- C5 pad 2: +3V3 -> /VOUT
- C6 pad 2: +3V3 -> /VOUT
- C7 pad 2: +3V3 -> /VOUT
- D1 pad 2: VBUS -> Net-(D1-A)
- D2 pad 1: +3V3 -> /VOUT
- D3 pad 1: +3V3 -> /VOUT
- D4 pad 1: +3V3 -> /VOUT
- D5 pad 1: +3V3 -> /VOUT
- J1 pad 1: unconnected-(J1-Pin_1-Pad1) -> /VOUT
- J1 pad 2: unconnected-(J1-Pin_2-Pad2) -> GND
- J1 pad 3: unconnected-(J1-Pin_3-Pad3) -> /SDA
- J1 pad 4: unconnected-(J1-Pin_4-Pad4) -> /SCL
- J4 pad 1: +3V3 -> /VOUT
- Q1 pad 1: VBUS -> Net-(D1-A)
- R1 pad 2: +3V3 -> /VOUT
- R2 pad 1: VBUS -> Net-(D1-A)
- R5 pad 2: +3V3 -> /VOUT
- SW1 pad 2: Net-(SW1-B) -> /VOUT
- U1 pad 2: +3V3 -> /VOUT
- U2 pad 1: Net-(SW1-B) -> VBUS
- U2 pad 3: Net-(SW1-B) -> VBUS
- U2 pad 5: +3V3 -> Net-(D1-A)
Routing:
- net VBUS: track 14.0 -> 24.2 mm
- net Net-(SW1-B): track 10.3 -> 0.00 mm
- net Net-(D1-A): track 0.00 -> 2.04 mm
- net +3V3: track 2.04 -> 0.00 mm
- added copper zone on F.Cu, net (none)
- added copper zone on F.Cu, net GND

Commit message: Update route and schematic
Parts:
- J5: value Conn_01x05 -> Serial_IN; footprint Connector_PinHeader_2.54mm:PinHeader_1x05_P2.54mm_Vertical -> Connector_PinHeader_2.54mm:PinHeader_1x03_P2.54mm_Vertical
- J6: value Conn_01x05 -> Serial_OUT; footprint Connector_PinHeader_2.54mm:PinHeader_1x05_P2.54mm_Vertical -> Connector_PinSocket_2.54mm:PinSocket_1x03_P2.54mm_Vertical
Connections:
- net /GPIO1 renamed /LEFT
- net /GPIO15 renamed /RIGHT
- C11 pad 2: /GPIO23 -> /DOWN
- C9 pad 2: /GPIO22 -> /UP
- J1 pad 5: unconnected-(J1-Pin_5-Pad5) -> /GPIO3
- J1 pad 6: unconnected-(J1-Pin_6-Pad6) -> /GPIO2
- J4 pad 1: /VOUT -> /SDA
- J4 pad 2: GND -> /SCL
- J4 pad 3: /SCL -> /VOUT
- J4 pad 4: /SDA -> GND
- J5 pad 1: unconnected-(J5-Pin_1-Pad1) -> /GPIO16
- J5 pad 2: unconnected-(J5-Pin_2-Pad2) -> /GPIO17
- J5 pad 3: unconnected-(J5-Pin_3-Pad3) -> GND
- J6 pad 1: unconnected-(J6-Pin_1-Pad1) -> /GPIO4
- J6 pad 2: unconnected-(J6-Pin_2-Pad2) -> /GPIO5
- J6 pad 3: unconnected-(J6-Pin_3-Pad3) -> GND
- R1 pad 1: /PIN -> Net-(U1-IO8)
- SW5 pad 2: /GPIO22 -> /DOWN
- SW7 pad 2: /GPIO23 -> /UP
- U1 pad 10: /PIN -> Net-(U1-IO8)
- U1 pad 11: unconnected-(U1-IO10-Pad11) -> /PIN
- U1 pad 20: /GPIO22 -> /UP
- U1 pad 21: /GPIO23 -> /DOWN
- U1 pad 24: /RX -> /GPIO17
- U1 pad 25: /TX -> /GPIO16
- U1 pad 26: unconnected-(U1-IO3-Pad26) -> /GPIO3
- U1 pad 27: unconnected-(U1-IO2-Pad27) -> /GPIO2
- U1 pad 4: unconnected-(U1-IO4-Pad4) -> /GPIO4
- U1 pad 5: unconnected-(U1-IO5-Pad5) -> /GPIO5
Routing:
- net /GPIO23: track 8.64 -> 0.00 mm
- net /DOWN: track 0.00 -> 8.64 mm
- net /UP: track 0.00 -> 8.63 mm
- net /GPIO22: track 8.63 -> 0.00 mm

Commit message: feat(Hw): Update route Community
Parts:
- F1: value 0.5A -> 0.75A
- SW4, SW6: value RESET -> ~
- moved C12 124.9 mm to (77.3, 165.3)
- moved D5 123.7 mm to (82.1, 165.4)
- moved D4 123.1 mm to (203.8, 142.5)
- moved C7 121.6 mm to (199.0, 142.3)
- moved C5 7.77 mm to (123.2, 39.8), turned to -90 degrees
- moved J6 7.62 mm to (71.4, 171.3), turned to -142.704 degrees
- moved J5 7.61 mm to (208.1, 152.4), turned to 130.491 degrees
- moved R6 7.23 mm to (118.1, 42.8)
- moved C2 6.12 mm to (191.7, 127.2), turned to 127.4 degrees
- moved U2 6.12 mm to (194.3, 125.4)
- moved C1 6.10 mm to (196.7, 123.7), turned to -52.6 degrees
- moved D1 3.41 mm to (199.6, 128.2)
- moved Q1 3.41 mm to (196.9, 130.3)
- moved R2 3.24 mm to (195.9, 127.3), turned to 37.4 degrees
- moved C13 2.78 mm to (97.6, 92.9), turned to 160 degrees
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Connections:
- C10 pad 2: /RIGHT -> /LEFT
- C11 pad 2: /DOWN -> /UP
- C8 pad 2: /LEFT -> /RIGHT
- C9 pad 2: /UP -> /DOWN
- SW4 pad 2: /LEFT -> /RIGHT
- SW6 pad 2: /RIGHT -> /LEFT
Routing:
- net /VOUT: track 0.00 -> 411.0 mm, vias 0 -> 15
- net /GPIO16: track 0.00 -> 148.1 mm, vias 0 -> 2
- net /GPIO17: track 0.00 -> 147.0 mm
- net Net-(D3-DOUT): track 0.00 -> 146.3 mm, vias 0 -> 4
- net Net-(D4-DOUT): track 0.00 -> 135.8 mm, vias 0 -> 2
- net /SDA: track 0.00 -> 114.7 mm, vias 0 -> 2
- net /SCL: track 0.00 -> 114.5 mm, vias 0 -> 2
- net /GPIO5: track 0.00 -> 96.0 mm, vias 0 -> 1
- net /GPIO4: track 0.00 -> 95.2 mm, vias 0 -> 1
- net /RIGHT: track 8.63 -> 94.7 mm
- net +BATT: track 0.00 -> 81.2 mm, vias 0 -> 1
- net /DOWN: track 8.64 -> 83.6 mm
- net /PIN: track 0.00 -> 74.9 mm
- net /LEFT: track 8.60 -> 70.0 mm, vias 0 -> 2
- net /GPIO3: track 0.00 -> 58.5 mm, vias 0 -> 1
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- added copper zone on B.Cu, net GND
