File: hardware/Bsides_2024_Sponsor/Bsides_2024_Sponsor.kicad_sch (KiCad schematic)
At the start: 44 parts, among them J1 Serial_IN, J2 Add_On, J3 OLED, J4 Serial_OUT, J5 Battery, J6 Battery, P1 USB_C_Plug_USB2.0, Q1 DMG3415U-7, SW1 ON, SW2 RESET, SW3 BOOT, SW4 RESET, SW6 RESET, U1 ESP32-C6-WROOM-1-N4, U2 AP2112K-3.3

Commit message: feat(Hw): Update BOM
Parts:
- C1, C10, C11, C12, C13, C14, C15, C2, C3, C4, C5, C6, C7, C8, C9, D1, Q1, R2, R5, R6, SW2, SW3, SW4, SW6: Proveedor Mouser -> JLCPCB
- D2, D3, D4, D5: Proveedor LCSC -> JLCPCB
- F1: value 0.5A -> 0.75A; LCSC# (none) -> C1972808; Proveedor Mouser -> JLCPCB
- J1: LCSC# (none) -> C5333416; Proveedor (none) -> JLCPCB
- J2: LCSC# (none) -> C5116527; Proveedor (none) -> JLCPCB
- J3: Proveedor (none) -> UNIT ELECTRONICS
- J4: LCSC# (none) -> C5116529; Proveedor (none) -> JLCPCB
- J5, J6: LCSC# C5290193 -> C5290181; Proveedor (none) -> JLCPCB y LCSC
- P1: LCSC# C2987386 -> C393939; Proveedor Mouser -> JLCPCB
- R1: LCSC# (none) -> C403480; Proveedor Mouser -> JLCPCB
- R3, R4: LCSC# C191782 -> C113390; Proveedor Mouser -> JLCPCB
- SW1: LCSC# - -> C431540; Proveedor Mouser -> JLCPCB; manf# JS102011SAQN -> (none)
- SW5, SW7: LCSC# C2886897 -> C318889; Proveedor Mouser -> JLCPCB
- U2: LCSC# C150742 -> C51118; Proveedor Mouser -> JLCPCB; manf# AP7365-33WG-7 -> AP2112K3.3TRG
Changed lines of the file:
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@@
 			)
 		)
-		(property "Proveedor" "LCSC"
+		(property "Proveedor" "JLCPCB"
 			(at 217.678 131.064 0)
 			(effects
@@
 			)
 		)
-		(property "Proveedor" "Mouser"
+		(property "Proveedor" "JLCPCB"
 			(at 274.574 118.999 0)
 			(effects
@@
 			)
 		)
-		(property "LCSC#" "C2886897"
+		(property "LCSC#" "C318889"
 			(at 257.683 65.278 0)
 			(effects
@@
 			)
 		)
-		(property "Proveedor" "Mouser"
+		(property "Proveedor" "JLCPCB"
 			(at 257.683 65.278 0)
 			(effects
@@
 			)
 		)
-		(property "LCSC#" ""
+		(property "LCSC#" "C403480"
 			(at 29.718 55.118 0)
 			(effects
@@
 			)
 		)
-		(property "Proveedor" "Mouser"
+		(property "Proveedor" "JLCPCB"
 			(at 29.718 55.118 0)
 			(effects
@@
 			)
 		)
-		(property "LCSC#" "C5290193"
+		(property "LCSC#" "C5290181"
 			(at 160.782 164.973 0)
 			(effects
@@
 			)
 		)
+		(property "Proveedor" "JLCPCB y LCSC"
+			(at 160.782 164.973 0)
+			(effects
+				(font
+					(size 1.27 1.27)
+				)
+				(hide yes)
+			)
+		)
 		(pin "1"
 		)
@@
 			)
 		)
+		(property "LCSC#" "C5116527"
+			(at 59.944 120.396 0)
+			(effects
+				(font
+					(size 1.27 1.27)
+				)
+				(hide yes)
+			)
+		)
+		(property "Proveedor" "JLCPCB"
+			(at 59.944 120.396 0)
+			(effects
+				(font
+					(size 1.27 1.27)
+				)
+				(hide yes)
+			)
+		)
 		(pin "1"
 		)
@@
 			)
 		)
-		(property "Proveedor" "Mouser"
+		(property "Proveedor" "JLCPCB"
 			(at 179.578 131.064 0)
 			(effects
@@
 			)
 		)
-		(property "Proveedor" "LCSC"
+		(property "Proveedor" "JLCPCB"
 			(at 192.278 131.064 0)
 			(effects
@@
 			)
 		)
+		(property "LCSC#" "C5333416"
+			(at 29.464 120.396 0)
+			(effects
+				(font
+					(size 1.27 1.27)
+				)
+				(hide yes)
+			)
+		)
+		(property "Proveedor" "JLCPCB"
+			(at 29.464 120.396 0)
+			(effects
+				(font
+					(size 1.27 1.27)
+				)
+				(hide yes)
+			)
+		)
 		(pin "2"
 		)
@@
 			)
 		)
-		(property "Proveedor" "Mouser"
+		(property "Proveedor" "JLCPCB"
 			(at 90.043 180.086 0)
 			(effects
@@
 			)
 		)
-		(property "Proveedor" "Mouser"
+		(property "Proveedor" "JLCPCB"
 			(at 169.418 34.036 0)
 			(effects
@@
 			)
 		)
-		(property "LCSC#" "C191782"
+		(property "LCSC#" "C113390"
 			(at 125.984 44.45 0)
 			(effects
@@
 			)
 		)
-		(property "Proveedor" "Mouser"
+		(property "Proveedor" "JLCPCB"
 			(at 125.984 44.45 0)
 			(effects
@@
 			)
 		)
-		(property "Proveedor" "LCSC"
+		(property "Proveedor" "JLCPCB"
 			(at 242.062 131.064 0)
 			(effects
@@
 			)
 		)
-		(property "Proveedor" "Mouser"
+		(property "Proveedor" "JLCPCB"
 			(at 54.356 178.308 0)
 			(effects
@@
 			)
 		)
-		(property "LCSC#" "-"
+		(property "LCSC#" "C431540"
 			(at 102.87 180.086 0)
 			(effects
@@
 			)
 		)
-		(property "manf#" "JS102011SAQN"
+		(property "manf#" ""
 			(at 102.87 180.086 0)
 			(effects
@@
 			)
 		)
-		(property "Proveedor" "Mouser"
+		(property "Proveedor" "JLCPCB"
 			(at 102.87 180.086 0)
 			(effects
@@
 			)
 		)
-		(property "Proveedor" "Mouser"
+		(property "Proveedor" "JLCPCB"
 			(at 15.494 85.217 0)
 			(effects
@@
 			)
 		)
+		(property "Proveedor" "UNIT ELECTRONICS"
+			(at 108.204 120.396 0)
+			(effects
+				(font
+					(size 1.27 1.27)
+				)
+				(hide yes)
+			)
+		)
 		(pin "1"
 		)
@@
 			)
 		)
+		(property "LCSC#" "C5116529"
+			(at 142.494 119.126 0)
+			(effects
+				(font
+					(size 1.27 1.27)
+				)
+				(hide yes)
+			)
+		)
+		(property "Proveedor" "JLCPCB"
+			(at 142.494 119.126 0)
+			(effects
+				(font
+					(size 1.27 1.27)
+				)
+				(hide yes)
+			)
+		)
 		(pin "2"
 		)
@@
 			)
 		)
-		(property "manf#" "AP7365-33WG-7"
+		(property "manf#" "AP2112K3.3TRG"
 			(at 69.088 176.276 0)
 			(effects
@@
 			)
 		)
-		(property "LCSC#" "C150742"
+		(property "LCSC#" "C51118"
 			(at 69.088 176.276 0)
 			(effects
@@
 			)
 		)
-		(property "Proveedor" "Mouser"
+		(property "Proveedor" "JLCPCB"
 			(at 69.088 176.276 0)
 			(effects
@@
 			)
 		)
-		(property "Proveedor" "Mouser"
+		(property "Proveedor" "JLCPCB"
 			(at 78.74 176.276 0)
 			(effects
@@
 			)
 		)
-		(property "Proveedor" "Mouser"
+		(property "Proveedor" "JLCPCB"
 			(at 259.969 52.07 0)
 			(effects
@@
 			)
 		)
-		(property "Proveedor" "Mouser"
+		(property "Proveedor" "JLCPCB"
 			(at 258.953 30.226 0)
 			(effects
@@
 			)
 		)
-		(property "Value" "0.5A"
+		(property "Value" "0.75A"
 			(at 127.254 36.9824 0)
 			(effects
@@
 			)
 		)
-		(property "LCSC#" ""
+		(property "LCSC#" "C1972808"
 			(at 127.254 39.37 0)
 			(effects
@@
 			)
 		)
-		(property "Proveedor" "Mouser"
+		(property "Proveedor" "JLCPCB"
 			(at 127.254 39.37 0)
 			(effects
@@
 			)
 		)
-		(property "Proveedor" "Mouser"
+		(property "Proveedor" "JLCPCB"
 			(at 23.114 85.09 0)
 			(effects
@@
 			)
 		)
-		(property "Proveedor" "Mouser"
+		(property "Proveedor" "JLCPCB"
 			(at 200.279 118.999 0)
 			(effects
@@
 			)
 		)
-		(property "Proveedor" "Mouser"
+		(property "Proveedor" "JLCPCB"
 			(at 169.418 47.752 0)
 			(effects
@@
 			)
 		)
-		(property "Proveedor" "Mouser"
+		(property "Proveedor" "JLCPCB"
 			(at 257.429 84.836 0)
 			(effects
@@
 			)
 		)
-		(property "LCSC#" "C2886897"
+		(property "LCSC#" "C318889"
 			(at 259.715 48.514 0)
 			(effects
@@
 			)
 		)
-		(property "Proveedor" "Mouser"
+		(property "Proveedor" "JLCPCB"
 			(at 259.715 48.514 0)
 			(effects
@@
 			)
 		)
-		(property "Proveedor" "Mouser"
+		(property "Proveedor" "JLCPCB"
 			(at 257.683 88.392 0)
 			(effects
@@
 			)
 		)
-		(property "Proveedor" "Mouser"
+		(property "Proveedor" "JLCPCB"
 			(at 257.937 68.834 0)
 			(effects
@@
 			)
 		)
-		(property "Proveedor" "Mouser"
+		(property "Proveedor" "JLCPCB"
 			(at 93.726 173.736 0)
 			(effects
@@
 			)
 		)
-		(property "LCSC#" "C191782"
+		(property "LCSC#" "C113390"
 			(at 125.984 46.99 0)
 			(effects
@@
 			)
 		)
-		(property "Proveedor" "Mouser"
+		(property "Proveedor" "JLCPCB"
 			(at 125.984 46.99 0)
 			(effects
@@
 			)
 		)
-		(property "Proveedor" "Mouser"
+		(property "Proveedor" "JLCPCB"
 			(at 249.682 118.999 0)
 			(effects
@@
 			)
 		)
-		(property "Proveedor" "Mouser"
+		(property "Proveedor" "JLCPCB"
 			(at 31.75 84.836 0)
 			(effects
@@
 			)
 		)
-		(property "LCSC#" "C5290193"
+		(property "LCSC#" "C5290181"
 			(at 160.782 159.766 0)
 			(effects
@@
 			)
 		)
+		(property "Proveedor" "JLCPCB y LCSC"
+			(at 160.782 159.766 0)
+			(effects
+				(font
+					(size 1.27 1.27)
+				)
+				(hide yes)
+			)
+		)
 		(pin "1"
 		)
@@
 			)
 		)
-		(property "Proveedor" "Mouser"
+		(property "Proveedor" "JLCPCB"
 			(at 225.171 118.999 0)
 			(effects
@@
 			)
 		)
-		(property "Proveedor" "Mouser"
+		(property "Proveedor" "JLCPCB"
 			(at 259.207 33.782 0)
 			(effects
@@
 			)
 		)
-		(property "Proveedor" "Mouser"
+		(property "Proveedor" "JLCPCB"
 			(at 169.545 36.068 0)
 			(effects
@@
 			)
 		)
-		(property "Proveedor" "Mouser"
+		(property "Proveedor" "JLCPCB"
 			(at 162.56 30.48 0)
 			(effects
@@
 			)
 		)
-		(property "LCSC#" "C2987386"
+		(property "LCSC#" "C393939"
 			(at 106.426 54.61 0)
 			(effects
@@
 			)
 		)
-		(property "Proveedor" "Mouser"
+		(property "Proveedor" "JLCPCB"
 			(at 106.426 54.61 0)
 			(effects
@@
 			)
 		)
-		(property "Proveedor" "Mouser"
+		(property "Proveedor" "JLCPCB"
 			(at 169.291 49.784 0)
 			(effects
@@
 			)
 		)
-		(property "Proveedor" "Mouser"
+		(property "Proveedor" "JLCPCB"
 			(at 83.058 186.817 0)
 			(effects
@@
 			)
 		)
-		(property "Proveedor" "LCSC"
+		(property "Proveedor" "JLCPCB"
 			(at 266.954 131.064 0)
 			(effects

Commit message: feat(Hw):Update_Labels_SCH_PCB_Sponsor_And_Staff
Connections:
- net GPIO1 renamed LEFT
- net GPIO15 renamed RIGHT
- net GPIO16 renamed TX
- net GPIO17 renamed RX
- net GPIO22 renamed UP
- net GPIO23 renamed DOWN
- net GPIO4 renamed RX1
- net GPIO5 renamed TX1
Changed lines of the file:
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@@
 		)
 	)
-	(label "GPIO15"
+	(label "RIGHT"
 		(at 70.104 68.58 0)
 		(fields_autoplaced yes)
@@
 		)
 	)
-	(label "GPIO17"
+	(label "RX"
 		(at 17.78 120.396 0)
 		(fields_autoplaced yes)
@@
 		)
 	)
-	(label "GPIO17"
+	(label "RX"
 		(at 70.104 65.786 0)
 		(fields_autoplaced yes)
@@
 		)
 	)
-	(label "GPIO5"
+	(label "TX1"
 		(at 131.826 119.126 0)
 		(fields_autoplaced yes)
@@
 		)
 	)
-	(label "GPIO16"
+	(label "TX"
 		(at 17.78 117.856 0)
 		(fields_autoplaced yes)
@@
 		)
 	)
-	(label "GPIO4"
+	(label "RX1"
 		(at 36.83 38.1 0)
 		(fields_autoplaced yes)
@@
 		)
 	)
-	(label "GPIO15"
+	(label "RIGHT"
 		(at 250.698 65.278 180)
 		(fields_autoplaced yes)
@@
 		)
 	)
-	(label "GPIO23"
+	(label "DOWN"
 		(at 251.968 48.514 180)
 		(fields_autoplaced yes)
@@
 		)
 	)
-	(label "GPIO1"
+	(label "LEFT"
 		(at 37.592 52.578 180)
 		(fields_autoplaced yes)
@@
 		)
 	)
-	(label "GPIO16"
+	(label "TX"
 		(at 70.104 62.992 0)
 		(fields_autoplaced yes)
@@
 		)
 	)
-	(label "GPIO22"
+	(label "UP"
 		(at 70.104 76.962 0)
 		(fields_autoplaced yes)
@@
 		)
 	)
-	(label "GPIO22"
+	(label "UP"
 		(at 251.206 30.226 180)
 		(fields_autoplaced yes)
@@
 		)
 	)
-	(label "GPIO23"
+	(label "DOWN"
 		(at 70.104 74.168 0)
 		(fields_autoplaced yes)
@@
 		)
 	)
-	(label "GPIO1"
+	(label "LEFT"
 		(at 250.19 84.836 180)
 		(fields_autoplaced yes)
@@
 		)
 	)
-	(label "GPIO4"
+	(label "RX1"
 		(at 131.826 116.586 0)
 		(fields_autoplaced yes)
@@
 		)
 	)
-	(label "GPIO5"
+	(label "TX1"
 		(at 36.83 41.148 0)
 		(fields_autoplaced yes)
