File: hardware/Bsides_2024_Staff/Bsides_2024_Staff.kicad_sch (KiCad schematic)
At the start: 44 parts, among them J1 Serial_IN, J2 Add_On, J3 OLED, J4 Serial_OUT, J5 Battery, J6 Battery, P1 USB_C_Plug_USB2.0, Q1 DMG3415U-7, SW1 ON, SW2 RESET, SW3 BOOT, SW4 RESET, SW6 RESET, U1 ESP32-C6-WROOM-1-N4, U2 AP2112K-3.3

Commit message: feat(Hw): Update BOM
Parts:
- C1: Proveedor Mouser -> JLCPCB; manf# TMK107BJ105KA8T -> (none)
- C10, C11, C12, C13, C14, C15, C6, C7, C8, C9: Proveedor Mouser -> JLCPCB; manf# KAM15AR71C104KM -> (none)
- C2, C3, C4, C5: Proveedor Mouser -> JLCPCB; manf# GRM188R61E106KA73J -> (none)
- D1: Proveedor Mouser -> JLCPCB; manf# MBR120LSFT1G -> (none)
- D2, D3, D4, D5: Proveedor LCSC -> JLCPCB
- F1: value 0.5A -> 0.75A; LCSC# (none) -> C1972808; Proveedor Mouser -> JLCPCB; manf# MFU0805FF00750P100 -> (none)
- J1: LCSC# (none) -> C5333416; Proveedor (none) -> JLCPCB
- J2: LCSC# (none) -> C5116527; Proveedor (none) -> JLCPCB
- J3: Proveedor (none) -> UNIT ELECTRONICS
- J4: LCSC# (none) -> C5116529; Proveedor (none) -> JLCPCB
- J5, J6: LCSC# C5290193 -> C5290181; Proveedor (none) -> JLCPCB y LCSC; manf# - -> (none)
- P1: LCSC# C2987386 -> C393939; Proveedor Mouser -> JLCPCB; manf# USB4105-GF-A -> (none)
- Q1: Proveedor Mouser -> JLCPCB; manf# DMG3415UQ-7 -> (none)
- R1: LCSC# (none) -> C403480; Proveedor Mouser -> JLCPCB; manf# ERJ-3GEYJ332V -> (none)
- R2: Proveedor Mouser -> JLCPCB; manf# RC0603DR-07100KL -> (none)
- R3, R4: LCSC# C191782 -> C113390; Proveedor Mouser -> JLCPCB; manf# AC0603DR-075K1L -> (none)
- R5: Proveedor Mouser -> JLCPCB; manf# RMC1/16K1002DTP -> (none)
- R6: Proveedor Mouser -> JLCPCB; manf# ERJ-3RBD4700V -> (none)
- SW1: LCSC# - -> C431540; Proveedor Mouser -> JLCPCB; manf# JS102011SAQN -> (none)
- SW2, SW3, SW4, SW6: Proveedor Mouser -> JLCPCB; manf# TL3342F160QG -> (none)
- SW5, SW7: LCSC# C2886897 -> C318889; Proveedor Mouser -> JLCPCB; manf# TL3342F160QG -> (none)
- U2: LCSC# C150742 -> C51118; Proveedor Mouser -> JLCPCB; manf# AP7365-33WG-7 -> (none)

Commit message: feat(Hw): Update schematic and route
Connections:
- net GPIO1 renamed LEFT
- net GPIO15 renamed RIGHT
- net GPIO16 renamed TX
- net GPIO17 renamed RX
- net GPIO22 renamed UP
- net GPIO23 renamed DOWN
- net GPIO4 renamed RX1
- net GPIO5 renamed TX1
Changed lines of the file:
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@@
 		)
 	)
-	(label "GPIO4"
+	(label "RX1"
 		(at 131.572 116.586 0)
 		(fields_autoplaced yes)
@@
 		)
 	)
-	(label "GPIO15"
+	(label "RIGHT"
 		(at 250.444 65.278 180)
 		(fields_autoplaced yes)
@@
 		)
 	)
-	(label "GPIO17"
+	(label "RX"
 		(at 17.526 120.396 0)
 		(fields_autoplaced yes)
@@
 		)
 	)
-	(label "GPIO1"
+	(label "LEFT"
 		(at 37.338 52.578 180)
 		(fields_autoplaced yes)
@@
 		)
 	)
-	(label "GPIO5"
+	(label "TX1"
 		(at 36.576 41.148 0)
 		(fields_autoplaced yes)
@@
 		)
 	)
-	(label "GPIO23"
+	(label "DOWN"
 		(at 251.714 48.514 180)
 		(fields_autoplaced yes)
@@
 		)
 	)
-	(label "GPIO23"
+	(label "DOWN"
 		(at 69.85 74.168 0)
 		(fields_autoplaced yes)
@@
 		)
 	)
-	(label "GPIO16"
+	(label "TX"
 		(at 69.85 62.992 0)
 		(fields_autoplaced yes)
@@
 		)
 	)
-	(label "GPIO22"
+	(label "UP"
 		(at 250.952 30.226 180)
 		(fields_autoplaced yes)
@@
 		)
 	)
-	(label "GPIO5"
+	(label "TX1"
 		(at 131.572 119.126 0)
 		(fields_autoplaced yes)
@@
 		)
 	)
-	(label "GPIO4"
+	(label "RX1"
 		(at 36.576 38.1 0)
 		(fields_autoplaced yes)
@@
 		)
 	)
-	(label "GPIO15"
+	(label "RIGHT"
 		(at 69.85 68.58 0)
 		(fields_autoplaced yes)
@@
 		)
 	)
-	(label "GPIO22"
+	(label "UP"
 		(at 69.85 76.962 0)
 		(fields_autoplaced yes)
@@
 		)
 	)
-	(label "GPIO1"
+	(label "LEFT"
 		(at 249.936 84.836 180)
 		(fields_autoplaced yes)
@@
 		)
 	)
-	(label "GPIO17"
+	(label "RX"
 		(at 69.85 65.786 0)
 		(fields_autoplaced yes)
@@
 		)
 	)
-	(label "GPIO16"
+	(label "TX"
 		(at 17.526 117.856 0)
 		(fields_autoplaced yes)
