File: hardware/Bsides_2024_ShittyAddon/Bsides_2024_ShittyAddon.kicad_pcb (KiCad board)
At the start: 2 copper layers, 49.7 x 25.4 mm, 13 parts, among them J1 SWD, J2 Conn_02x03_Odd_Even, U1 PY32F002AA15M6TU

Commit message: feat(Hw):Update_Shitty_Add_On
Parts:
- added kibuzzard-666C77E0: G***, kibuzzard-666C77E0, B.Cu at (145.7, 78.0)
- added kibuzzard-666C77E0: G***, kibuzzard-666C77E0, B.Cu at (129.8, 68.8)
- added kibuzzard-666C7809: G***, kibuzzard-666C7809, B.Cu at (153.9, 74.2)
- added kibuzzard-666C7809: G***, kibuzzard-666C7809, B.Cu at (129.8, 73.6)
- added kibuzzard-666C7823: G***, kibuzzard-666C7823, B.Cu at (139.3, 73.7)
- added kibuzzard-666C7874: G***, kibuzzard-666C7874, B.Cu at (151.4, 75.3)
- added kibuzzard-666C787C: G***, kibuzzard-666C787C, B.Cu at (148.7, 76.5)

Commit message: feat(hw): add logos shitty addon
Parts:
- added G***: LOGO, Aesthetics:electronic_cats_logo_8x6, B.Cu at (145.1, 71.5)
- added G***: LOGO, LOGO, B.Cu at (122.5, 73.7)
- added REF**: OSHW-Logo_7.5x8mm_SilkScreen, Symbol:OSHW-Logo_7.5x8mm_SilkScreen, B.Cu at (82.6, 103.4)

Commit message: feat(Hw): Update label ShittyAddon
Parts:
- turned kibuzzard-666C7809 to -155 degrees
Changed lines of the file:
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@@
 				(font
 					(size 0.001 0.001)
+					(thickness 0.15)
 				)
 				(justify mirror)
@@
 				(font
 					(size 0.001 0.001)
+					(thickness 0.15)
 				)
 				(justify mirror)
@@
 				(font
 					(size 1.27 1.27)
+					(thickness 0.15)
 				)
 				(justify mirror)
@@
 				(font
 					(size 1.27 1.27)
+					(thickness 0.15)
 				)
 				(justify mirror)
@@
 				(font
 					(size 1.27 1.27)
+					(thickness 0.15)
 				)
 				(justify mirror)
@@
 				(font
 					(size 0.001 0.001)
+					(thickness 0.15)
 				)
 				(justify mirror)
@@
 				(font
 					(size 0.001 0.001)
+					(thickness 0.15)
 				)
 				(justify mirror)
@@
 		(tags "resistor")
 		(property "Reference" "R2"
-			(at 3.095527 -0.639856 -70)
+			(at 3.095527 -0.639857 -70)
 			(layer "B.SilkS")
 			(effects
@@
 	(footprint "kibuzzard-666C7809"
 		(layer "B.Cu")
-		(at 153.93 74.15 25)
+		(at 153.93 74.15 -155)
 		(descr "Generated with KiBuzzard")
 		(tags "kb_params=eyJBbGlnbm1lbnRDaG9pY2UiOiAiQ2VudGVyIiwgIkNhcExlZnRDaG9pY2UiOiAiKCIsICJDYXBSaWdodENob2ljZSI6ICIpIiwgIkZvbnRDb21ib0JveCI6ICJVYnVudHVNb25vLUIiLCAiSGVpZ2h0Q3RybCI6IDAuNywgIkxheWVyQ29tYm9Cb3giOiAiRi5TaWxrUyIsICJMaW5lU3BhY2luZ0N0cmwiOiAxLjUsICJNdWx0aUxpbmVUZXh0IjogIkdORCIsICJQYWRkaW5nQm90dG9tQ3RybCI6IDEuMCwgIlBhZGRpbmdMZWZ0Q3RybCI6IDIuNSwgIlBhZGRpbmdSaWdodEN0cmwiOiAyLjUsICJQYWRkaW5nVG9wQ3RybCI6IDEuMCwgIldpZHRoQ3RybCI6IDAuNywgImFkdmFuY2VkQ2hlY2tib3giOiBmYWxzZSwgImlubGluZUZvcm1hdFRleHRib3giOiBmYWxzZSwgImxpbmVvdmVyU3R5bGVDaG9pY2UiOiAiU3F1YXJlIiwgImxpbmVvdmVyVGhpY2tuZXNzQ3RybCI6IDF9")
@@
 				(font
 					(size 1.27 1.27)
+					(thickness 0.15)
 				)
 				(justify mirror)
@@
 				(font
 					(size 1.27 1.27)
+					(thickness 0.15)
 				)
 				(justify mirror)
@@
 				(font
 					(size 1.27 1.27)
+					(thickness 0.15)
 				)
 				(justify mirror)
@@
 				(font
 					(size 0.001 0.001)
+					(thickness 0.15)
 				)
 				(justify mirror)
@@
 				(font
 					(size 0.001 0.001)
+					(thickness 0.15)
 				)
 				(justify mirror)
@@
 				(font
 					(size 1.27 1.27)
+					(thickness 0.15)
 				)
 				(justify mirror)
@@
 				(font
 					(size 1.27 1.27)
+					(thickness 0.15)
 				)
 				(justify mirror)
@@
 				(font
 					(size 1.27 1.27)
+					(thickness 0.15)
 				)
 				(justify mirror)
@@
 				(font
 					(size 0.001 0.001)
+					(thickness 0.15)
 				)
 				(justify mirror)
@@
 				(font
 					(size 0.001 0.001)
+					(thickness 0.15)
 				)
 				(justify mirror)
@@
 				(font
 					(size 0.001 0.001)
+					(thickness 0.15)
 				)
 				(justify mirror)
@@
 				(font
 					(size 0.001 0.001)
+					(thickness 0.15)
 				)
 				(justify mirror)
